Commit message: updated gitignore with tfrecord files. Added cnn_learner_detached. Fixed issue #1. Added several new maps.

File: src/robots/sim/atrv.urdf (robot description, URDF)
Before this commit: robot artv, 2 links, 1 joints
Links:
- removed link laser
- added link base_scan
Joints:
- removed joint base_laser
- added joint joint_laser: type fixed, parent base_link, child base_scan, origin xyz=0 0 0.3 rpy=0 0 0
